File: Porthole Controller/Porthole Controller.kicad_pcb (KiCad board)
At the start: 2 copper layers, 65 x 65 mm, 19 parts, among them J1 STRIP1, J2 STRIP2, J3 STRIP3, J4 STRIP4, J5 INMP441, J6 Conn_02x04_Top_Bottom, J7 - +, J8 Conn_01x04, U1 113991054, U2 SN74AHCT125DR

Commit message: Added Rev 1 Gerber Files for PCB order
Other:
- board text added: "The Magpie's Nest WLED Controller, Rev 1 Design By Peter Spierenburg and Mike Matthews 2024-06-01"
Changed lines of the file:
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@@
 			(outputformat 1)
 			(mirror no)
-			(drillshape 1)
+			(drillshape 0)
 			(scaleselection 1)
-			(outputdirectory "")
+			(outputdirectory "./rev1")
 		)
 	)
@@
 		)
 		(fp_text user "${REFERENCE}"
-			(at -1.27 2.54 270)
+			(at -1.27 2.54 -90)
 			(layer "F.Fab")
 			(effects
@@
 		(tags "Resistor Axial_DIN0204 series Axial Horizontal pin pitch 5.08mm 0.167W length 3.6mm diameter 1.6mm")
 		(property "Reference" "R3"
-			(at 2.54 -1.92 270)
+			(at 2.54 -1.92 -90)
 			(layer "F.SilkS")
 			(effects
@@
 		)
 		(property "Value" "100"
-			(at 2.54 1.92 270)
+			(at 2.54 1.92 -90)
 			(layer "F.SilkS")
 			(effects
@@
 		)
 		(fp_text user "${REFERENCE}"
-			(at 2.54 0 270)
+			(at 2.54 0 -90)
 			(layer "F.Fab")
 			(effects
@@
 		(tags "SN74AHC125NG4 ")
 		(property "Reference" "U2"
-			(at 3.81 20 0)
+			(at 3.839 16.1306 0)
 			(unlocked yes)
 			(layer "F.SilkS")
@@
 		(tags "C Disc series Radial pin pitch 2.50mm  diameter 3.0mm width 1.6mm Capacitor")
 		(property "Reference" "C1"
-			(at -2.5 0 270)
+			(at -2.5 0 -90)
 			(layer "F.SilkS")
 			(effects
@@
 		)
 		(property "Value" "100nF"
-			(at 1.25 2.05 270)
+			(at 1.25 2.05 -90)
 			(layer "F.SilkS")
 			(effects
@@
 		)
 		(fp_text user "${REFERENCE}"
-			(at 1.25 0 270)
+			(at 1.25 0 -90)
 			(layer "F.Fab")
 			(effects
@@
 		(tags "Resistor Axial_DIN0204 series Axial Horizontal pin pitch 5.08mm 0.167W length 3.6mm diameter 1.6mm")
 		(property "Reference" "R4"
-			(at 2.54 -1.92 270)
+			(at 2.54 -1.92 -90)
 			(layer "F.SilkS")
 			(effects
@@
 		)
 		(property "Value" "100"
-			(at 2.54 1.92 270)
+			(at 2.54 1.92 -90)
 			(layer "F.SilkS")
 			(effects
@@
 		)
 		(fp_text user "${REFERENCE}"
-			(at 2.54 0 270)
+			(at 2.54 0 -90)
 			(layer "F.Fab")
 			(effects
@@
 		)
 	)
+	(gr_text "The Magpie's Nest WLED Controller, Rev 1\nDesign By Peter Spierenburg and Mike Matthews\n2024-06-01"
+		(at 143.3322 106.0196 90)
+		(layer "F.SilkS")
+		(effects
+			(font
+				(size 1 1)
+				(thickness 0.1)
+			)
+			(justify bottom)
+		)
+	)

Commit message: Updated footprints
Parts:
- C2, C3, C4, C5: footprint Capacitor_THT:CP_Radial_D6.3mm_P2.50mm -> Capacitor_THT:CP_Radial_D8.0mm_P3.80mm
- moved R4 6.54 mm to (176.5, 125.7)
- moved J4 6.53 mm to (171.4, 133.3)
- moved C5 6.46 mm to (171.4, 123.2)
- moved J5 6.34 mm to (193.0, 127.0), turned to 0 degrees
- moved R3 3.80 mm to (156.2, 125.7)
- moved J3 3.71 mm to (151.1, 133.3)
- moved C4 3.64 mm to (151.1, 123.2)
- moved J8 3.25 mm to (194.3, 95.3)
- moved J6 3.18 mm to (194.3, 92.7)
- moved J7 1.32 mm to (190.5, 81.3)
- moved J1 1.23 mm to (175.3, 81.3)
- moved J2 1.22 mm to (157.5, 81.3)
- moved R2 1.11 mm to (152.4, 88.9)
- moved R1 1.10 mm to (170.2, 88.9)
- moved C2 1.08 mm to (175.3, 91.4)
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Connections:
- J5 pad 3: WS -> 3.3V
- J5 pad 4: 3.3V -> WS
- J5 pad 5: SCK -> SD
- J5 pad 6: SD -> SCK
- U1 pad 10: SCK -> WS
- U1 pad 9: WS -> SCK
Routing:
- net 5V: track 192.3 -> 185.4 mm
- net Net-(U2-4Y): track 16.1 -> 22.7 mm
- net SCK: track 13.9 -> 20.0 mm
- net SD: track 13.9 -> 19.6 mm
- net D5: track 6.52 -> 10.3 mm
- net D4: track 6.52 -> 10.3 mm
- net D3: track 33.8 -> 31.0 mm
- net Net-(U2-3Y): track 9.40 -> 11.5 mm
- net D0: track 5.45 -> 7.40 mm
- net D1: track 5.45 -> 7.40 mm
- net D2: track 26.5 -> 25.1 mm
- net D6: track 29.6 -> 28.4 mm
- net WS: track 17.5 -> 16.4 mm
- net D7: track 19.1 -> 18.6 mm
